File: hardware/main/gate_drive.kicad_sch (KiCad schematic)
At the start: 17 parts, among them Q1 IRLZ44N, Q2 IRLZ44N, U5 ADUM3223ARZ

Commit message: added setup files for stm32
Parts:
- C4: value 4.7u -> 10u
Changed lines of the file:
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@@
 			)
 		)
-		(property "Value" "4.7u"
+		(property "Value" "10u"
 			(at 67.056 91.44 0)
 			(show_name no)
