File: hardware/main/power_mgmt.kicad_sch (KiCad schematic)
At the start: 19 parts, among them Q7 DMP6050SSD, Q9 DMP6050SSD, U12 AP2112K-2.6

Commit message: added status LED's to schema, fixed gate drive error, added BOM
Parts:
- added D10, D7, D8, D9: LED, LED_SMD:LED_0603_1608Metric, symbol Device:LED
- added R43: 680, Resistor_SMD:R_0603_1608Metric_Pad0.98x0.95mm_HandSolder, symbol Device:R
- added R44: 100, Resistor_SMD:R_0603_1608Metric_Pad0.98x0.95mm_HandSolder, symbol Device:R
- added R45: 6.98k, Resistor_SMD:R_1206_3216Metric_Pad1.30x1.75mm_HandSolder, symbol Device:R
- added R46: 3k, Resistor_SMD:R_0805_2012Metric_Pad1.20x1.40mm_HandSolder, symbol Device:R
- C26, C27, C30, C31: footprint Capacitor_SMD:C_0603_1608Metric_Pad1.08x0.95mm_HandSolder -> Capacitor_SMD:C_0603_1608Metric
- C28, C29: footprint (none) -> footprint:PCAP_12_5x20-THRU-ELECT_NCA
- R17, R4: footprint (none) -> Resistor_SMD:R_0603_1608Metric
- TP21, TP22, TP23: footprint (none) -> TestPoint:TestPoint_Keystone_5015_Micro_Mini
Connections:
- net +12V: now also R46.1
- net +24V: now also R45.1
- net +3.3V: now also R44.1
- net GNDA: now also D10.1 (K), D7.1 (K), D8.1 (K), D9.1 (K)
- net 5V_STATUS_LED: now reaches C30.1, D5.1 (K), U12.1 (VIN), U12.3 (EN)
- net 5V_STATUS_LED: now also R43.1
- new net: D7.2 (A), R43.2
- new net: D9.2 (A), R45.2
- new net: D8.2 (A), R44.2
- new net: D10.2 (A), R46.2
Other:
- note added: "STATUS INDICATORS"
- note removed: "TODO: Add status indicators"
- note removed: "The PMOS on the bootstrap and DC Bus are reverse voltage polarity protection."
- moved on the sheet: C30, C31, CR3, D5, D6, Q9A, R17, TP22, TP23, U12

Commit message: footprints updated in hardware
Parts:
- R43, R44: footprint Resistor_SMD:R_0603_1608Metric_Pad0.98x0.95mm_HandSolder -> Resistor_SMD:R_0603_1608Metric
- R45: footprint Resistor_SMD:R_1206_3216Metric_Pad1.30x1.75mm_HandSolder -> Resistor_SMD:R_1206_3216Metric
- R46: footprint Resistor_SMD:R_0805_2012Metric_Pad1.20x1.40mm_HandSolder -> Resistor_SMD:R_0805_2012Metric
Changed lines of the file:
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@@
 			)
 		)
-		(property "Footprint" "Resistor_SMD:R_1206_3216Metric_Pad1.30x1.75mm_HandSolder"
+		(property "Footprint" "Resistor_SMD:R_1206_3216Metric"
 			(at 63.5 85.598 90)
 			(hide yes)
@@
 			)
 		)
-		(property "Footprint" "Resistor_SMD:R_0603_1608Metric_Pad0.98x0.95mm_HandSolder"
+		(property "Footprint" "Resistor_SMD:R_0603_1608Metric"
 			(at 64.77 132.588 90)
 			(hide yes)
@@
 			)
 		)
-		(property "Footprint" "Resistor_SMD:R_0805_2012Metric_Pad1.20x1.40mm_HandSolder"
+		(property "Footprint" "Resistor_SMD:R_0805_2012Metric"
 			(at 63.5 107.188 90)
 			(hide yes)
@@
 			)
 		)
-		(property "Footprint" "Resistor_SMD:R_0603_1608Metric_Pad0.98x0.95mm_HandSolder"
+		(property "Footprint" "Resistor_SMD:R_0603_1608Metric"
 			(at 64.77 142.748 90)
 			(hide yes)

Commit message: hardware layout started
Parts:
- removed Q7, Q9: DMP6050SSD, Package_SO:SOIC-8_3.9x4.9mm_P1.27mm, symbol Transistor_FET:DMP6050SSD
- removed TP22: Keystone 5015, TestPoint:TestPoint_Keystone_5015_Micro_Mini, symbol Connector:TestPoint_Alt
- added Q7, Q8: SSM3J351R, footprint:SSM3J351R, symbol Simulation_SPICE:PMOS
Connections:
- net +12V: now also Q8.3 (S)
- net +24V: now also Q7.3 (S)
- net 12V_EXT: now also Q8.1 (D)
- net 24V_EXT: now also Q7.1 (D)
- net at D4.2 (A), R4.1: now also Q7.2 (G)
- net at D6.2 (A), R17.1: now also Q8.2 (G)
Changed lines of the file:
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@@
 	)
 	(junction
-		(at 207.01 104.14)
-		(diameter 0)
-		(color 0 0 0 0)
-	)
-	(junction
 		(at 194.31 129.54)
 		(diameter 0)
@@
 	(wire
 		(pts
-			(xy 207.01 104.14) (xy 214.63 104.14)
-		)
-		(stroke
-			(width 0)
-			(type default)
-		)
-	)
-	(wire
-		(pts
 			(xy 199.39 44.45) (xy 209.55 44.45)
 		)
@@
 	(wire
 		(pts
-			(xy 152.4 104.14) (xy 207.01 104.14)
+			(xy 152.4 104.14) (xy 214.63 104.14)
 		)
 		(stroke
@@
 	)
 	(symbol
-		(lib_id "Connector:TestPoint_Alt")
-		(at 207.01 104.14 180)
+		(lib_id "Simulation_SPICE:PMOS")
+		(at 209.55 34.29 270)
+		(mirror x)
 		(unit 1)
 		(body_style 1)
@@
 		(dnp no)
 		(fields_autoplaced yes)
-		(property "Reference" "TP22"
-			(at 209.55 106.1719 0)
+		(property "Reference" "Q7"
+			(at 209.55 25.4 90)
 			(show_name no)
 			(do_not_autoplace no)
@@
 					(size 1.27 1.27)
 				)
-				(justify right)
 			)
 		)
-		(property "Value" "Keystone 5015"
-			(at 209.55 108.7119 0)
+		(property "Value" "SSM3J351R"
+			(at 209.55 27.94 90)
 			(show_name no)
 			(do_not_autoplace no)
@@
 					(size 1.27 1.27)
 				)
-				(justify right)
 			)
 		)
-		(property "Footprint" "TestPoint:TestPoint_Keystone_5015_Micro_Mini"
-			(at 201.93 104.14 0)
+		(property "Footprint" "footprint:SSM3J351R"
+			(at 212.09 29.21 0)
 			(hide yes)
 			(show_name no)
@@
 			)
 		)
-		(property "Datasheet" ""
-			(at 201.93 104.14 0)
+		(property "Datasheet" "https://ngspice.sourceforge.io/docs/ngspice-html-manual/manual.xhtml#cha_MOSFETs"
+			(at 196.85 34.29 0)
 			(hide yes)
 			(show_name no)
@@
 			)
 		)
-		(property "Description" "test point (alternative shape)"
-			(at 207.01 104.14 0)
+		(property "Description" "P-MOSFET transistor, drain/source/gate"
+			(at 209.55 34.29 0)
+			(hide yes)
+			(show_name no)
+			(do_not_autoplace no)
+			(effects
+				(font
+					(size 1.27 1.27)
+				)
+			)
+		)
+		(property "Sim.Device" "PMOS"
+			(at 192.405 34.29 0)
+			(hide yes)
+			(show_name no)
+			(do_not_autoplace no)
+			(effects
+				(font
+					(size 1.27 1.27)
+				)
+			)
+		)
+		(property "Sim.Type" "VDMOS"
+			(at 190.5 34.29 0)
+			(hide yes)
+			(show_name no)
+			(do_not_autoplace no)
+			(effects
+				(font
+					(size 1.27 1.27)
+				)
+			)
+		)
+		(property "Sim.Pins" "1=D 2=G 3=S"
+			(at 194.31 34.29 0)
 			(hide yes)
 			(show_name no)
@@
 		(pin "1"
 		)
+		(pin "2"
+		)
+		(pin "3"
+		)
 		(instances
 			(project "mosfets"
 				(path "/6b82a8a8-ae2c-4987-9dc0-17eac5149d3f/5ced536b-3314-4fa5-ab67-f1b42cff0312"
-					(reference "TP22")
+					(reference "Q7")
 					(unit 1)
 				)
@@
 	)
 	(symbol
-		(lib_name "DMP6050SSD_1")
-		(lib_id "Transistor_FET:DMP6050SSD")
-		(at 214.63 82.55 90)
+		(lib_id "Simulation_SPICE:PMOS")
+		(at 214.63 82.55 270)
+		(mirror x)
 		(unit 1)
 		(body_style 1)
@@
 		(dnp no)
 		(fields_autoplaced yes)
-		(property "Reference" "Q9"
+		(property "Reference" "Q8"
 			(at 214.63 73.66 90)
 			(show_name no)
@@
 			)
 		)
-		(property "Value" "DMP6050SSD"
+		(property "Value" "SSM3J351R"
 			(at 214.63 76.2 90)
 			(show_name no)
@@
 			)
 		)
-		(property "Footprint" "Package_SO:SOIC-8_3.9x4.9mm_P1.27mm"
-			(at 216.535 77.47 0)
+		(property "Footprint" "footprint:SSM3J351R"
+			(at 217.17 77.47 0)
 			(hide yes)
 			(show_name no)
@@
 				(font
 					(size 1.27 1.27)
-					(italic yes)
 				)
-				(justify left)
 			)
 		)
-		(property "Datasheet" "https://www.diodes.com/assets/Datasheets/DMP6050SSD.pdf"
-			(at 218.44 77.47 0)
+		(property "Datasheet" "https://ngspice.sourceforge.io/docs/ngspice-html-manual/manual.xhtml#cha_MOSFETs"
+			(at 201.93 82.55 0)
 			(hide yes)
 			(show_name no)
@@
 					(size 1.27 1.27)
 				)
-				(justify left)
 			)
 		)
-		(property "Description" "-11.3A Id, -60V Vds, P-Channel Power MOSFET, 55mOhm Ron, 11.9nC Qg (typ), SO-8"
+		(property "Description" "P-MOSFET transistor, drain/source/gate"
 			(at 214.63 82.55 0)
 			(hide yes)
@@
 			)
 		)
-		(pin "2"
-		)
-		(pin "5"
-		)
-		(pin "8"
-		)
-		(pin "4"
-		)
-		(pin "1"
-		)
-		(pin "3"
-		)
-		(pin "6"
-		)
-		(pin "7"
-		)
-		(instances
-			(project "mosfets"
-				(path "/6b82a8a8-ae2c-4987-9dc0-17eac5149d3f/5ced536b-3314-4fa5-ab67-f1b42cff0312"
-					(reference "Q9")
-					(unit 1)
-				)
-			)
-		)
-	)
-	(symbol
-		(lib_name "DMP6050SSD_1")
-		(lib_id "Transistor_FET:DMP6050SSD")
-		(at 209.55 34.29 90)
-		(unit 1)
-		(body_style 1)
-		(exclude_from_sim no)
-		(in_bom yes)
-		(on_board yes)
-		(in_pos_files yes)
-		(dnp no)
-		(fields_autoplaced yes)
-		(property "Reference" "Q7"
-			(at 209.55 25.4 90)
-			(show_name no)
-			(do_not_autoplace no)
-			(effects
-				(font
-					(size 1.27 1.27)
-				)
-			)
-		)
-		(property "Value" "DMP6050SSD"
-			(at 209.55 27.94 90)
-			(show_name no)
-			(do_not_autoplace no)
-			(effects
-				(font
-					(size 1.27 1.27)
-				)
-			)
-		)
-		(property "Footprint" "Package_SO:SOIC-8_3.9x4.9mm_P1.27mm"
-			(at 211.455 29.21 0)
+		(property "Sim.Device" "PMOS"
+			(at 197.485 82.55 0)
 			(hide yes)
 			(show_name no)
@@
 				(font
 					(size 1.27 1.27)
-					(italic yes)
 				)
-				(justify left)
 			)
 		)
-		(property "Datasheet" "https://www.diodes.com/assets/Datasheets/DMP6050SSD.pdf"
-			(at 213.36 29.21 0)
+		(property "Sim.Type" "VDMOS"
+			(at 195.58 82.55 0)
 			(hide yes)
 			(show_name no)
@@
 					(size 1.27 1.27)
 				)
-				(justify left)
 			)
 		)
-		(property "Description" "-11.3A Id, -60V Vds, P-Channel Power MOSFET, 55mOhm Ron, 11.9nC Qg (typ), SO-8"
-			(at 209.55 34.29 0)
+		(property "Sim.Pins" "1=D 2=G 3=S"
+			(at 199.39 82.55 0)
 			(hide yes)
 			(show_name no)
@@
 			)
 		)
-		(pin "2"
-		)
-		(pin "5"
-		)
-		(pin "8"
-		)
-		(pin "4"
-		)
 		(pin "1"
 		)
-		(pin "3"
-		)
-		(pin "6"
+		(pin "2"
 		)
-		(pin "7"
+		(pin "3"
 		)
 		(instances
 			(project "mosfets"
 				(path "/6b82a8a8-ae2c-4987-9dc0-17eac5149d3f/5ced536b-3314-4fa5-ab67-f1b42cff0312"
-					(reference "Q7")
+					(reference "Q8")
 					(unit 1)
 				)
