File: hardware/main/power_mgmt.kicad_sch (KiCad schematic)
At the start: 26 parts, among them Q7 SSM3J351R, Q8 SSM3J351R, U12 AP2112K-2.6

Commit message: added setup files for stm32
Parts:
- added NT1: NetTie_2, symbol Device:NetTie_2
Connections:
- net GNDA: now also NT1.1; no longer C26.2, C27.2, C28.2, C29.2, CR1.2, CR3.2, D10.1 (K), D9.1 (K), R17.2, R4.2, TP21.1
- new net GNDPWR: C26.2, C27.2, C28.2, C29.2, CR1.2, CR3.2, D10.1 (K), D9.1 (K), NT1.2, R17.2, R4.2, TP21.1
Changed lines of the file:
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@@
+	)
+	(junction
+		(at 142.24 55.88)
+		(diameter 0)
+		(color 0 0 0 0)
+	)
+	(junction
+		(at 152.4 129.54)
+		(diameter 0)
+		(color 0 0 0 0)
+	)
+	(junction
+		(at 134.62 31.75)
+		(diameter 0)
+		(color 0 0 0 0)
+	)
+	(junction
+		(at 224.79 31.75)
+		(diameter 0)
+		(color 0 0 0 0)
 	)
 	(junction
@@
 	)
 	(junction
-		(at 142.24 55.88)
-		(diameter 0)
-		(color 0 0 0 0)
-	)
-	(junction
-		(at 152.4 129.54)
-		(diameter 0)
-		(color 0 0 0 0)
-	)
-	(junction
-		(at 134.62 31.75)
-		(diameter 0)
-		(color 0 0 0 0)
-	)
-	(junction
-		(at 224.79 31.75)
-		(diameter 0)
-		(color 0 0 0 0)
-	)
-	(junction
 		(at 139.7 31.75)
 		(diameter 0)
@@
 	(wire
 		(pts
+			(xy 85.09 26.67) (xy 90.17 26.67)
+		)
+		(stroke
+			(width 0)
+			(type default)
+		)
+	)
+	(wire
+		(pts
 			(xy 177.8 41.91) (xy 177.8 31.75)
 		)
@@
 	(wire
 		(pts
+			(xy 95.25 26.67) (xy 99.06 26.67)
+		)
+		(stroke
+			(width 0)
+			(type default)
+		)
+	)
+	(wire
+		(pts
 			(xy 214.63 87.63) (xy 214.63 92.71)
 		)
@@
 	(wire
 		(pts
-			(xy 104.14 26.67) (xy 85.09 26.67)
-		)
-		(stroke
-			(width 0)
-			(type default)
-		)
-	)
-	(wire
-		(pts
 			(xy 166.37 31.75) (xy 177.8 31.75)
 		)
@@
 	(wire
 		(pts
-			(xy 104.14 31.75) (xy 104.14 26.67)
+			(xy 99.06 31.75) (xy 99.06 26.67)
 		)
 		(stroke
@@
 	(symbol
 		(lib_id "power:GNDPWR")
-		(at 104.14 31.75 0)
+		(at 99.06 31.75 0)
 		(unit 1)
 		(body_style 1)
@@
 		(fields_autoplaced yes)
 		(property "Reference" "#PWR029"
-			(at 104.14 36.83 0)
+			(at 99.06 36.83 0)
 			(hide yes)
 			(show_name no)
@@
 		)
 		(property "Value" "GNDPWR"
-			(at 104.013 35.56 0)
+			(at 98.933 35.56 0)
 			(show_name no)
 			(do_not_autoplace no)
@@
 		)
 		(property "Footprint" ""
-			(at 104.14 33.02 0)
+			(at 99.06 33.02 0)
 			(hide yes)
 			(show_name no)
@@
 		)
 		(property "Datasheet" ""
-			(at 104.14 33.02 0)
+			(at 99.06 33.02 0)
 			(hide yes)
 			(show_name no)
@@
 		)
 		(property "Description" "Power symbol creates a global label with name \"GNDPWR\" , global ground"
-			(at 104.14 31.75 0)
+			(at 99.06 31.75 0)
 			(hide yes)
 			(show_name no)
@@
 					(unit 1)
 				)
+			)
+		)
+	)
+	(symbol
+		(lib_id "Device:NetTie_2")
+		(at 92.71 26.67 0)
+		(unit 1)
+		(body_style 1)
+		(exclude_from_sim no)
+		(in_bom no)
+		(on_board yes)
+		(in_pos_files yes)
+		(dnp no)
+		(fields_autoplaced yes)
+		(property "Reference" "NT1"
+			(at 92.71 21.59 0)
+			(show_name no)
+			(do_not_autoplace no)
+			(effects
+				(font
+					(size 1.27 1.27)
+				)
+			)
+		)
+		(property "Value" "NetTie_2"
+			(at 92.71 24.13 0)
+			(show_name no)
+			(do_not_autoplace no)
+			(effects
+				(font
+					(size 1.27 1.27)
+				)
+			)
+		)
+		(property "Footprint" ""
+			(at 92.71 26.67 0)
+			(hide yes)
+			(show_name no)
+			(do_not_autoplace no)
+			(effects
+				(font
+					(size 1.27 1.27)
+				)
+			)
+		)
+		(property "Datasheet" ""
+			(at 92.71 26.67 0)
+			(hide yes)
+			(show_name no)
+			(do_not_autoplace no)
+			(effects
+				(font
+					(size 1.27 1.27)
+				)
+			)
+		)
+		(property "Description" "Net tie, 2 pins"
+			(at 92.71 26.67 0)
+			(hide yes)
+			(show_name no)
+			(do_not_autoplace no)
+			(effects
+				(font
+					(size 1.27 1.27)
+				)
+			)
+		)
+		(pin "1"
+		)
+		(pin "2"
+		)
+		(instances
+			(project "mosfets"
+				(path "/6b82a8a8-ae2c-4987-9dc0-17eac5149d3f/5ced536b-3314-4fa5-ab67-f1b42cff0312"
+					(reference "NT1")
+					(unit 1)
+				)
