File: hardware/main/mosfets.kicad_pcb (KiCad board)
At the start: 4 copper layers, 142 parts, among them J1 Screw_Terminal_01x03, J2 Screw_Terminal_01x02, J3 Screw_Terminal_01x02, J4 Screw_Terminal_01x02, J5 Conn_01x08_Pin, J6 Conn_02x19_Odd_Even, J7 Conn_02x19_Odd_Even, Q1 IRLZ44N, Q2 IRLZ44N, Q3 IRLZ44N, Q4 IRLZ44N, Q5 IRLZ44N, Q6 IRLZ44N, Q7 SSM3J351R, Q8 SSM3J351R, U10 TL331, U11 TL331, U12 AP2112K-2.6, U13 74LVC1G332, U2 INA181, U3 INA181, U4 INA181, U5 ADUM3223ARZ, U6 ADUM3223ARZ, U7 ADUM3223ARZ, U8 LMV321, U9 TL331

Commit message: added setup files for stm32
Parts:
- removed TP10, TP7: TestPoint, TestPoint:TestPoint_Pad_D1.5mm
- removed TP23: Keystone 5015, TestPoint:TestPoint_Keystone_5015_Micro_Mini
- C4, C5, C9: value 4.7u -> 10u
- U12: value AP2112K-2.6 -> AP2112K-3.3
- moved R15 214.0 mm to (179.2, 124.5), turned to -90 degrees
- moved J4 87.7 mm to (140.8, 27.1), turned to 180 degrees
- moved U9 82.5 mm to (166.0, 52.2)
- moved U4 81.1 mm to (172.5, 125.6), turned to -90 degrees
- moved C15 77.5 mm to (172.5, 121.8)
- moved C20 77.1 mm to (161.8, 52.0), turned to -90 degrees
- moved U2 74.5 mm to (168.6, 61.4), turned to -90 degrees
- moved R18 74.4 mm to (169.8, 57.3), turned to 90 degrees
- moved C16 73.8 mm to (171.1, 64.1), turned to -90 degrees
- moved C18 73.3 mm to (169.5, 125.6), turned to 90 degrees
- moved R5 72.5 mm to (169.0, 52.2), turned to -90 degrees
- moved U3 71.5 mm to (169.2, 92.5), turned to -90 degrees
- moved C13 70.8 mm to (168.1, 57.3), turned to -90 degrees
- moved U10 70.7 mm to (165.0, 81.2)
- moved R13 69.3 mm to (181.8, 60.8), turned to 180 degrees
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Connections:
- C26 pad 2: GNDA -> GNDPWR
- C27 pad 2: GNDA -> GNDPWR
- C28 pad 2: GNDA -> GNDPWR
- C29 pad 2: GNDA -> GNDPWR
- CR1 pad 2: GNDA -> GNDPWR
- CR3 pad 2: GNDA -> GNDPWR
- D10 pad 1: GNDA -> GNDPWR
- D9 pad 1: GNDA -> GNDPWR
- J2 pad 1: GNDA -> GNDPWR
- J3 pad 1: GNDA -> GNDPWR
- R13 pad 2: GNDA -> GNDPWR
- R14 pad 2: GNDA -> GNDPWR
- R15 pad 2: GNDA -> GNDPWR
- R17 pad 2: GNDA -> GNDPWR
- R24 pad 1: /OCP_Current_Sens/VSHUNT_B_P -> /OCP_Current_Sens/V_REF
- R27 pad 1: /OCP_Current_Sens/VSHUNT_C_P -> /OCP_Current_Sens/V_REF
- R4 pad 2: GNDA -> GNDPWR
- TP21 pad 1: GNDA -> GNDPWR
- U10 pad 3: /OCP_Current_Sens/V_REF -> /OCP_Current_Sens/VSHUNT_B_P
- U11 pad 3: /OCP_Current_Sens/V_REF -> /OCP_Current_Sens/VSHUNT_C_P
- U2 pad 4: GNDA -> GNDPWR
- U3 pad 4: GNDA -> GNDPWR
- U4 pad 4: GNDA -> GNDPWR
Routing:
- net /PHASE_A: track 29.4 -> 0.00 mm
- net /OCP_Current_Sens/VSHUNT_A_P: track 18.0 -> 1.41 mm
- net Net-(U5-VOA): track 12.6 -> 0.00 mm
- net Net-(U5-VOB): track 12.3 -> 0.11 mm
- net Net-(U5-VDDA): track 6.82 -> 0.00 mm
- net +12V: track 14.9 -> 9.60 mm
- net Net-(D1-K): track 3.81 -> 0.00 mm
- net Net-(Q2-G): track 2.99 -> 0.00 mm
- net Net-(Q1-G): track 2.68 -> 0.00 mm
- net GNDA: track 17.3 -> 16.0 mm
- net GNDPWR: track 0.00 -> 1.23 mm
