File: hardware/PWM_6_step_SWPWM/PWM_6_step_SWPWM_DIRTY.kicad_sch (KiCad schematic)
At the start: 8 parts, among them J3 Screw_Terminal_01x02, J4 Conn_01x06_Pin, J5 Screw_Terminal_01x03

Commit message: fixes to PCB
Connections:
- no-connect marks 4 -> 0
